File: CoreBoard_Rev1/CoreBoard_Rev1.kicad_pcb (KiCad board)
At the start: 2 copper layers, 135.1 x 84.3 mm, 93 parts, among them J1 RJ45_LED_Shielded, SW1 SW_Push, SW10 SW_Push, SW11 SW_Push, SW12 SW_Push, SW13 SW_Push, SW14 SW_Push, SW15 SW_Push, SW16 SW_SPDT, SW2 SW_Push, SW3 SW_Push, SW4 SW_Push, SW5 SW_Push, SW6 SW_Push, SW7 SW_Push, SW8 SW_Push, SW9 SW_Push, U1 Teensy4.1_DEV-16771, U3 SHHD003A0A, U4 74HC148, U5 74HC148, U6 74HC00, U7 OKI

Commit message: Gerbs Generated
Parts:
- C2: footprint Capacitor_SMD:C_0603_1608Metric_Pad1.08x0.95mm_HandSolder -> Capacitor_SMD:C_1206_3216Metric_Pad1.33x1.80mm_HandSolder
- moved C2 1.68 mm to (182.0, 98.3), turned to 0 degrees
- moved C3 0.76 mm to (183.8, 101.9)
- moved U7 0.51 mm to (186.3, 105.4)
Routing:
- net PV: track 77.0 -> 74.3 mm
- net +3V3: track 531.9 -> 530.6 mm
- net B8: track 87.1 -> 86.6 mm
- net B15: track 83.0 -> 82.5 mm
- net GND: vias 30 -> 31

Commit message: Gerbs Generated
Parts:
- moved C1 2.54 mm to (92.2, 89.8)
Routing:
- net Net-(C1-Pad2): track 26.0 -> 23.4 mm
Changed lines of the file:
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@@
   )
   (footprint "Capacitor_SMD:C_0603_1608Metric_Pad1.08x0.95mm_HandSolder" (layer "F.Cu")
-    (at 94.742 89.7625 90)
+    (at 92.202 89.7636 90)
     (descr "Capacitor SMD 0603 (1608 Metric), square (rectangular) end terminal, IPC_7351 nominal with elongated pad for handsoldering. (Body size source: IPC-SM-782 page 76, https://www.pcb-3d.com/wordpress/wp-content/uploads/ipc-sm-782a_amendment_1_and_2.pdf), generated with kicad-footprint-generator")
     (tags "capacitor handsolder")
@@
     (property "ki_keywords" "cap capacitor")
     (attr smd)
-    (fp_text reference "C1" (at -2.8945 0.254) (layer "F.SilkS")
+    (fp_text reference "C1" (at -2.4638 0.127) (layer "F.SilkS")
         (effects (font (size 1 1) (thickness 0.15)))
     )
@@
   (via (at 89.281 80.01) (size 0.8) (drill 0.4) (layers "F.Cu" "B.Cu") (free) (net 1))
   (segment (start 83.003 83.765) (end 84.328 85.09) (width 0.25) (layer "F.Cu") (net 2))
+  (segment (start 86.900563 88.9) (end 92.2009 88.9) (width 0.25) (layer "F.Cu") (net 2))
   (segment (start 86.900563 88.9) (end 85.630563 87.63) (width 0.25) (layer "F.Cu") (net 2))
   (segment (start 85.630563 86.392563) (end 84.328 85.09) (width 0.25) (layer "F.Cu") (net 2))
   (segment (start 83.933 77.865) (end 83.003 78.795) (width 0.25) (layer "F.Cu") (net 2))
   (segment (start 86.868 80.01) (end 84.723 77.865) (width 0.25) (layer "F.Cu") (net 2))
-  (segment (start 94.742 88.9) (end 86.900563 88.9) (width 0.25) (layer "F.Cu") (net 2))
   (segment (start 83.003 78.795) (end 83.003 83.765) (width 0.25) (layer "F.Cu") (net 2))
   (segment (start 84.328 85.09) (end 84.328 83.82) (width 0.25) (layer "F.Cu") (net 2))

Commit message: Layout Edits
Parts:
- moved C1 0.89 mm to (91.4, 89.3), turned to 180 degrees
- moved R35 0.51 mm to (153.2, 94.7)
- moved D20 0.47 mm to (155.2, 94.7)
Routing:
- net PV: track 74.3 -> 71.8 mm
- net +3V3: track 530.6 -> 529.5 mm, vias 9 -> 11
- net Net-(C1-Pad2): track 23.4 -> 22.4 mm
- net ReverseSW: track 96.5 -> 97.1 mm
- net +5V: vias 1 -> 5
- net NeoPixels: vias 0 -> 2
Other:
- board text removed: "Servo 1-3"
- board text removed: "Servo 4-6"
- board text removed: "Servo 7-9"
