File: board/accelerometer.kicad_sch (KiCad schematic)
At the start: 1 part, among them U4 GY-521

Commit message: Layout edits
Parts:
- U4: footprint GY-521:GY-521 -> CoreBoard:GY-521
Changed lines of the file:
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@@
 			)
 		)
-		(property "Footprint" "GY-521:GY-521"
+		(property "Footprint" "CoreBoard:GY-521"
 			(at 60.96 53.34 0)
 			(effects
