File: board/led_decoder.kicad_sch (KiCad schematic)
At the start: 34 parts, among them Q1 AO3401A, Q10 AO3401A, Q12 AO3401A, Q2 AO3401A, Q3 AO3401A, Q4 AO3401A, Q5 AO3401A, Q6 AO3401A, Q7 AO3401A, Q8 AO3401A, Q9 AO3401A, U1 74VHC138FT

Commit message: rev2 progress
Connections:
- net +3.3V: now also Q10.2 (S), Q12.2 (S), Q7.2 (S), Q8.2 (S), Q9.2 (S); no longer Q10.3 (D), Q12.3 (D), Q7.3 (D), Q8.3 (D), Q9.3 (D)
- net BL_EN: now also Q5.2 (S); no longer Q5.3 (D)
- net BR_EN: now also Q3.2 (S); no longer Q3.3 (D)
- net FL_EN: now also Q6.2 (S); no longer Q6.3 (D)
- net FR_EN: now also Q1.2 (S); no longer Q1.3 (D)
- net ML_EN: now also Q4.2 (S); no longer Q4.3 (D)
- net MR_EN: now also Q2.2 (S); no longer Q2.3 (D)
- net at D4.2 (A): now also Q5.3 (D); no longer Q5.2 (S)
- net at D15.2 (A): now also Q12.3 (D); no longer Q12.2 (S)
- net at D13.2 (A): now also Q6.3 (D); no longer Q6.2 (S)
- net at D5.2 (A): now also Q3.3 (D); no longer Q3.2 (S)
- net at D12.2 (A): now also Q2.3 (D); no longer Q2.2 (S)
- net at D6.2 (A): now also Q4.3 (D); no longer Q4.2 (S)
- net at D18.2 (A): now also Q10.3 (D); no longer Q10.2 (S)
- net at D8.2 (A): now also Q1.3 (D); no longer Q1.2 (S)
- net at D16.2 (A): now also Q8.3 (D); no longer Q8.2 (S)
- net at D14.2 (A): now also Q9.3 (D); no longer Q9.2 (S)
- net at D17.2 (A): now also Q7.3 (D); no longer Q7.2 (S)
Changed lines of the file:
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@@
 		(lib_id "Transistor_FET:AO3401A")
 		(at 224.79 97.79 0)
+		(mirror x)
 		(unit 1)
 		(exclude_from_sim no)
@@
 		(dnp no)
 		(property "Reference" "Q5"
-			(at 231.14 96.5199 0)
+			(at 231.14 99.0601 0)
 			(effects
 				(font
@@
 		)
 		(property "Value" "AO3401A"
-			(at 231.14 99.0599 0)
+			(at 231.14 96.5201 0)
 			(effects
 				(font
@@
 		)
 		(property "Footprint" "Package_TO_SOT_SMD:SOT-23"
-			(at 229.87 99.695 0)
+			(at 229.87 95.885 0)
 			(effects
 				(font
@@
 		)
 		(property "Datasheet" "http://www.aosmd.com/pdfs/datasheet/AO3401A.pdf"
-			(at 229.87 101.6 0)
+			(at 229.87 93.98 0)
 			(effects
 				(font
@@
 		(lib_id "Transistor_FET:AO3401A")
 		(at 182.88 96.52 0)
+		(mirror x)
 		(unit 1)
 		(exclude_from_sim no)
@@
 		(dnp no)
 		(property "Reference" "Q6"
-			(at 189.23 95.2499 0)
+			(at 189.23 97.7901 0)
 			(effects
 				(font
@@
 		)
 		(property "Value" "AO3401A"
-			(at 189.23 97.7899 0)
+			(at 189.23 95.2501 0)
 			(effects
 				(font
@@
 		)
 		(property "Footprint" "Package_TO_SOT_SMD:SOT-23"
-			(at 187.96 98.425 0)
+			(at 187.96 94.615 0)
 			(effects
 				(font
@@
 		)
 		(property "Datasheet" "http://www.aosmd.com/pdfs/datasheet/AO3401A.pdf"
-			(at 187.96 100.33 0)
+			(at 187.96 92.71 0)
 			(effects
 				(font
@@
 		(lib_id "Transistor_FET:AO3401A")
 		(at 220.98 36.83 0)
+		(mirror x)
 		(unit 1)
 		(exclude_from_sim no)
@@
 		(dnp no)
 		(property "Reference" "Q2"
-			(at 227.33 35.5599 0)
+			(at 227.33 38.1001 0)
 			(effects
 				(font
@@
 		)
 		(property "Value" "AO3401A"
-			(at 227.33 38.0999 0)
+			(at 227.33 35.5601 0)
 			(effects
 				(font
@@
 		)
 		(property "Footprint" "Package_TO_SOT_SMD:SOT-23"
-			(at 226.06 38.735 0)
+			(at 226.06 34.925 0)
 			(effects
 				(font
@@
 		)
 		(property "Datasheet" "http://www.aosmd.com/pdfs/datasheet/AO3401A.pdf"
-			(at 226.06 40.64 0)
+			(at 226.06 33.02 0)
 			(effects
 				(font
@@
 		(lib_id "Transistor_FET:AO3401A")
 		(at 80.01 137.16 0)
+		(mirror x)
 		(unit 1)
 		(exclude_from_sim no)
@@
 		(dnp no)
 		(property "Reference" "Q12"
-			(at 86.36 135.8899 0)
+			(at 86.36 138.4301 0)
 			(effects
 				(font
@@
 		)
 		(property "Value" "AO3401A"
-			(at 86.36 138.4299 0)
+			(at 86.36 135.8901 0)
 			(effects
 				(font
@@
 		)
 		(property "Footprint" "Package_TO_SOT_SMD:SOT-23"
-			(at 85.09 139.065 0)
+			(at 85.09 135.255 0)
 			(effects
 				(font
@@
 		)
 		(property "Datasheet" "http://www.aosmd.com/pdfs/datasheet/AO3401A.pdf"
-			(at 85.09 140.97 0)
+			(at 85.09 133.35 0)
 			(effects
 				(font
@@
 		(lib_id "Transistor_FET:AO3401A")
 		(at 44.45 80.01 0)
+		(mirror x)
 		(unit 1)
 		(exclude_from_sim no)
@@
 		(dnp no)
 		(property "Reference" "Q10"
-			(at 50.8 78.7399 0)
+			(at 50.8 81.2801 0)
 			(effects
 				(font
@@
 		)
 		(property "Value" "AO3401A"
-			(at 50.8 81.2799 0)
+			(at 50.8 78.7401 0)
 			(effects
 				(font
@@
 		)
 		(property "Footprint" "Package_TO_SOT_SMD:SOT-23"
-			(at 49.53 81.915 0)
+			(at 49.53 78.105 0)
 			(effects
 				(font
@@
 		)
 		(property "Datasheet" "http://www.aosmd.com/pdfs/datasheet/AO3401A.pdf"
-			(at 49.53 83.82 0)
+			(at 49.53 76.2 0)
 			(effects
 				(font
@@
 		(lib_id "Transistor_FET:AO3401A")
 		(at 259.08 96.52 0)
+		(mirror x)
 		(unit 1)
 		(exclude_from_sim no)
@@
 		(dnp no)
 		(property "Reference" "Q4"
-			(at 265.43 95.2499 0)
+			(at 265.43 97.7901 0)
 			(effects
 				(font
@@
 		)
 		(property "Value" "AO3401A"
-			(at 265.43 97.7899 0)
+			(at 265.43 95.2501 0)
 			(effects
 				(font
@@
 		)
 		(property "Footprint" "Package_TO_SOT_SMD:SOT-23"
-			(at 264.16 98.425 0)
+			(at 264.16 94.615 0)
 			(effects
 				(font
@@
 		)
 		(property "Datasheet" "http://www.aosmd.com/pdfs/datasheet/AO3401A.pdf"
-			(at 264.16 100.33 0)
+			(at 264.16 92.71 0)
 			(effects
 				(font
@@
 		(lib_id "Transistor_FET:AO3401A")
 		(at 113.03 137.16 0)
+		(mirror x)
 		(unit 1)
 		(exclude_from_sim no)
@@
 		(dnp no)
 		(property "Reference" "Q8"
-			(at 119.38 135.8899 0)
+			(at 119.38 138.4301 0)
 			(effects
 				(font
@@
 		)
 		(property "Value" "AO3401A"
-			(at 119.38 138.4299 0)
+			(at 119.38 135.8901 0)
 			(effects
 				(font
@@
 		)
 		(property "Footprint" "Package_TO_SOT_SMD:SOT-23"
-			(at 118.11 139.065 0)
+			(at 118.11 135.255 0)
 			(effects
 				(font
@@
 		)
 		(property "Datasheet" "http://www.aosmd.com/pdfs/datasheet/AO3401A.pdf"
-			(at 118.11 140.97 0)
+			(at 118.11 133.35 0)
 			(effects
 				(font
@@
 		(lib_id "Transistor_FET:AO3401A")
 		(at 44.45 138.43 0)
+		(mirror x)
 		(unit 1)
 		(exclude_from_sim no)
@@
 		(dnp no)
 		(property "Reference" "Q9"
-			(at 50.8 137.1599 0)
+			(at 50.8 139.7001 0)
 			(effects
 				(font
@@
 		)
 		(property "Value" "AO3401A"
-			(at 50.8 139.6999 0)
+			(at 50.8 137.1601 0)
 			(effects
 				(font
@@
 		)
 		(property "Footprint" "Package_TO_SOT_SMD:SOT-23"
-			(at 49.53 140.335 0)
+			(at 49.53 136.525 0)
 			(effects
 				(font
@@
 		)
 		(property "Datasheet" "http://www.aosmd.com/pdfs/datasheet/AO3401A.pdf"
-			(at 49.53 142.24 0)
+			(at 49.53 134.62 0)
 			(effects
 				(font
@@
 		(lib_id "Transistor_FET:AO3401A")
 		(at 254 36.83 0)
+		(mirror x)
 		(unit 1)
 		(exclude_from_sim no)
@@
 		(dnp no)
 		(property "Reference" "Q3"
-			(at 260.35 35.5599 0)
+			(at 260.35 38.1001 0)
 			(effects
 				(font
@@
 		)
 		(property "Value" "AO3401A"
-			(at 260.35 38.0999 0)
+			(at 260.35 35.5601 0)
 			(effects
 				(font
@@
 		)
 		(property "Footprint" "Package_TO_SOT_SMD:SOT-23"
-			(at 259.08 38.735 0)
+			(at 259.08 34.925 0)
 			(effects
 				(font
@@
 		)
 		(property "Datasheet" "http://www.aosmd.com/pdfs/datasheet/AO3401A.pdf"
-			(at 259.08 40.64 0)
+			(at 259.08 33.02 0)
 			(effects
 				(font
@@
 		(lib_id "Transistor_FET:AO3401A")
 		(at 182.88 36.83 0)
+		(mirror x)
 		(unit 1)
 		(exclude_from_sim no)
@@
 		(dnp no)
 		(property "Reference" "Q1"
-			(at 189.23 35.5599 0)
+			(at 189.23 38.1001 0)
 			(effects
 				(font
@@
 		)
 		(property "Value" "AO3401A"
-			(at 189.23 38.0999 0)
+			(at 189.23 35.5601 0)
 			(effects
 				(font
@@
 		)
 		(property "Footprint" "Package_TO_SOT_SMD:SOT-23"
-			(at 187.96 38.735 0)
+			(at 187.96 34.925 0)
 			(effects
 				(font
@@
 		)
 		(property "Datasheet" "http://www.aosmd.com/pdfs/datasheet/AO3401A.pdf"
-			(at 187.96 40.64 0)
+			(at 187.96 33.02 0)
 			(effects
 				(font
@@
 		(lib_id "Transistor_FET:AO3401A")
 		(at 149.86 138.43 0)
+		(mirror x)
 		(unit 1)
 		(exclude_from_sim no)
@@
 		(dnp no)
 		(property "Reference" "Q7"
-			(at 156.21 137.1599 0)
+			(at 156.21 139.7001 0)
 			(effects
 				(font
@@
 		)
 		(property "Value" "AO3401A"
-			(at 156.21 139.6999 0)
+			(at 156.21 137.1601 0)
 			(effects
 				(font
@@
 		)
 		(property "Footprint" "Package_TO_SOT_SMD:SOT-23"
-			(at 154.94 140.335 0)
+			(at 154.94 136.525 0)
 			(effects
 				(font
@@
 		)
 		(property "Datasheet" "http://www.aosmd.com/pdfs/datasheet/AO3401A.pdf"
-			(at 154.94 142.24 0)
+			(at 154.94 134.62 0)
 			(effects
 				(font
