File: core_board/Connectors.kicad_sch (KiCad schematic)
At the start: 12 parts, among them J10 Conn_01x04_Pin, J11 Conn_01x04_Pin, J12 Conn_01x04_Pin, J3 Conn_01x04_Pin, J4 Conn_01x04_Pin, J5 Conn_01x04_Pin, J6 Conn_01x04_Pin, J7 Conn_01x02_Pin, J9 Conn_01x02_Pin

Commit message: Finish Schematic
Parts:
- added J14, J15: Conn_01x04_Pin, Connector:Tag-Connect_TC2030-IDC-FP_2x03_P1.27mm_Vertical, symbol Connector:Conn_01x04_Pin
- added Q10, Q11, Q12, Q13, Q14, Q9: BSS138, Package_TO_SOT_SMD:SOT-23, symbol Transistor_FET:BSS138
- added R22, R23, R24, R25, R26, R27: 10K, Package_TO_SOT_SMD:SOT-23, symbol Device:R_US
Connections:
- net GND: now also Q10.2 (S), Q11.2 (S), Q12.2 (S), Q13.2 (S), Q14.2 (S), Q9.2 (S), R22.2, R23.2, R24.2, R25.2, R26.2, R27.2
- new net: J15.2 (Pin_2), Q13.3 (D)
- new net: J14.1 (Pin_1), Q11.3 (D)
- new net: J14.2 (Pin_2), Q10.3 (D)
- new net: J14.3 (Pin_3), Q9.3 (D)
- new net: J15.1 (Pin_1), Q14.3 (D)
- new net: J15.3 (Pin_3), Q12.3 (D)
- new net +5V: J14.4 (Pin_4), J15.4 (Pin_4)
- new net BLUE_PWM_Internal: Q11.1 (G), R24.1
- new net BLUE_PWM_StateDisplay: Q14.1 (G), R27.1
- new net GREEN_PWM_Internal: Q10.1 (G), R23.1
- new net GREEN_PWM_StateDisplay: Q13.1 (G), R26.1
- new net RED_PWM_Internal: Q9.1 (G), R22.1
- new net RED_PWM_StateDisplay: Q12.1 (G), R25.1
Other:
- moved on the sheet: J10, J11, J12, R18, R19, R20

Commit message: Fix fan connectors
Parts:
- removed J10, J11, J12: Conn_01x04_Pin, Package_DFN_QFN:QFN-20-1EP_5x5mm_P0.65mm_EP3.35x3.35mm, symbol Connector:Conn_01x04_Pin
- removed R18, R19, R20: 10K, Package_DIP:DIP-8_W7.62mm, symbol Device:R_US
- added J10, J11, J8: Conn_01x02_Pin, Converter_DCDC:Converter_DCDC_Cyntec_MUN12AD01-SH, symbol Connector:Conn_01x02_Pin
- added Q15, Q16, Q17: NMOS, Package_DFN_QFN:SiliconLabs_QFN-20-1EP_3x3mm_P0.5mm, symbol Simulation_SPICE:NMOS
- added R28, R30, R32: 100, RF_Module:ESP32-S2-WROVER, symbol Device:R_US
- added R29, R31, R33: 10k, RF_Module:ESP32-S2-WROVER, symbol Device:R_US
Connections:
- net +24V: now also J10.2 (Pin_2), J11.2 (Pin_2), J8.2 (Pin_2)
- net FanPWM1: now also R28.1
- net FanPWM2: now also R30.1
- net FanPWM3: now also R32.1
- net GND: now also Q15.3 (S), Q16.3 (S), Q17.3 (S), R29.1, R31.1, R33.1
- new net: Q16.2 (G), R30.2, R31.2
- new net: J8.1 (Pin_1), Q15.1 (D)
- new net: Q15.2 (G), R28.2, R29.2
- new net: J10.1 (Pin_1), Q16.1 (D)
- new net: J11.1 (Pin_1), Q17.1 (D)
- new net: Q17.2 (G), R32.2, R33.2

Commit message: Pull down resisters
Parts:
- added J12: Conn_01x02_Pin, Package_DFN_QFN:QFN-20-1EP_5x5mm_P0.65mm_EP3.35x3.35mm, symbol Connector:Conn_01x02_Pin
Connections:
- new net CANHigh2: J12.2 (Pin_2)
- new net CANLow2: J12.1 (Pin_1)
Other:
- moved on the sheet: J7
Changed lines of the file:
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@@
 	(wire
 		(pts
-			(xy 226.06 40.64) (xy 231.14 40.64)
+			(xy 203.2 39.37) (xy 208.28 39.37)
 		)
 		(stroke
@@
 	(wire
 		(pts
-			(xy 226.06 43.18) (xy 231.14 43.18)
+			(xy 203.2 41.91) (xy 208.28 41.91)
 		)
 		(stroke
@@
 	(wire
 		(pts
+			(xy 248.92 39.37) (xy 254 39.37)
+		)
+		(stroke
+			(width 0)
+			(type default)
+		)
+	)
+	(wire
+		(pts
 			(xy 125.73 52.07) (xy 128.27 52.07)
 		)
@@
 	(wire
 		(pts
+			(xy 248.92 41.91) (xy 254 41.91)
+		)
+		(stroke
+			(width 0)
+			(type default)
+		)
+	)
+	(wire
+		(pts
 			(xy 144.78 92.71) (xy 144.78 91.44)
 		)
@@
 		)
 	)
+	(hierarchical_label "CANHigh2"
+		(shape bidirectional)
+		(at 248.92 39.37 180)
+		(effects
+			(font
+				(size 1.27 1.27)
+			)
+			(justify right)
+		)
+	)
 	(hierarchical_label "LeftPan"
 		(shape input)
@@
 	(hierarchical_label "CANLow"
 		(shape bidirectional)
-		(at 226.06 43.18 180)
+		(at 203.2 41.91 180)
 		(effects
 			(font
@@
 	(hierarchical_label "CANHigh"
 		(shape bidirectional)
-		(at 226.06 40.64 180)
+		(at 203.2 39.37 180)
 		(effects
 			(font
@@
 		)
 	)
+	(hierarchical_label "CANLow2"
+		(shape bidirectional)
+		(at 248.92 41.91 180)
+		(effects
+			(font
+				(size 1.27 1.27)
+			)
+			(justify right)
+		)
+	)
 	(hierarchical_label "Spare1"
 		(shape input)
@@
 	)
 	(symbol
+		(lib_id "Connector:Conn_01x02_Pin")
+		(at 259.08 41.91 180)
+		(unit 1)
+		(body_style 1)
+		(exclude_from_sim no)
+		(in_bom yes)
+		(on_board yes)
+		(in_pos_files yes)
+		(dnp no)
+		(fields_autoplaced yes)
+		(property "Reference" "J12"
+			(at 260.35 39.3699 0)
+			(show_name no)
+			(do_not_autoplace no)
+			(effects
+				(font
+					(size 1.27 1.27)
+				)
+				(justify right)
+			)
+		)
+		(property "Value" "Conn_01x02_Pin"
+			(at 260.35 41.9099 0)
+			(show_name no)
+			(do_not_autoplace no)
+			(effects
+				(font
+					(size 1.27 1.27)
+				)
+				(justify right)
+			)
+		)
+		(property "Footprint" "Package_DFN_QFN:QFN-20-1EP_5x5mm_P0.65mm_EP3.35x3.35mm"
+			(at 259.08 41.91 0)
+			(hide yes)
+			(show_name no)
+			(do_not_autoplace no)
+			(effects
+				(font
+					(size 1.27 1.27)
+				)
+			)
+		)
+		(property "Datasheet" ""
+			(at 259.08 41.91 0)
+			(hide yes)
+			(show_name no)
+			(do_not_autoplace no)
+			(effects
+				(font
+					(size 1.27 1.27)
+				)
+			)
+		)
+		(property "Description" "Generic connector, single row, 01x02, script generated"
+			(at 259.08 41.91 0)
+			(hide yes)
+			(show_name no)
+			(do_not_autoplace no)
+			(effects
+				(font
+					(size 1.27 1.27)
+				)
+			)
+		)
+		(pin "1"
+		)
+		(pin "2"
+		)
+		(instances
+			(project "core_board"
+				(path "/e01d6047-065c-44c8-9643-8ab57e6ffae6/1e3ab302-e360-416c-88e3-133e033fb1f0"
+					(reference "J12")
+					(unit 1)
+				)
+			)
+		)
+	)
+	(symbol
 		(lib_id "Device:R_US")
 		(at 261.62 142.24 0)
@@
 	(symbol
 		(lib_id "Connector:Conn_01x02_Pin")
-		(at 236.22 43.18 180)
+		(at 213.36 41.91 180)
 		(unit 1)
 		(body_style 1)
@@
 		(fields_autoplaced yes)
 		(property "Reference" "J7"
-			(at 237.49 40.6399 0)
+			(at 214.63 39.3699 0)
 			(show_name no)
 			(do_not_autoplace no)
@@
 		)
 		(property "Value" "Conn_01x02_Pin"
-			(at 237.49 43.1799 0)
+			(at 214.63 41.9099 0)
 			(show_name no)
 			(do_not_autoplace no)
@@
 		)
 		(property "Footprint" "Package_DFN_QFN:QFN-20-1EP_5x5mm_P0.65mm_EP3.35x3.35mm"
-			(at 236.22 43.18 0)
+			(at 213.36 41.91 0)
 			(hide yes)
 			(show_name no)
@@
 		)
 		(property "Datasheet" ""
-			(at 236.22 43.18 0)
+			(at 213.36 41.91 0)
 			(hide yes)
 			(show_name no)
@@
 		)
 		(property "Description" "Generic connector, single row, 01x02, script generated"
-			(at 236.22 43.18 0)
+			(at 213.36 41.91 0)
 			(hide yes)
 			(show_name no)

Commit message: finish stuff
Parts:
- added R38, R39, R40, R41: 220, RF_Module:ESP32-S2-WROVER, symbol Device:R_US
Connections:
- net +7.5V: now also R38.2, R39.2, R40.2, R41.2; no longer J3.4 (Pin_4), J4.4 (Pin_4), J5.4 (Pin_4), J6.4 (Pin_4)
- new net: J3.4 (Pin_4), R40.1
- new net: J5.4 (Pin_4), R38.1
- new net: J4.4 (Pin_4), R39.1
- new net: J6.4 (Pin_4), R41.1

Commit message: add
Parts:
- added Q24: NMOS, Package_DFN_QFN:SiliconLabs_QFN-20-1EP_3x3mm_P0.5mm, symbol Simulation_SPICE:NMOS
- added R34: 100, RF_Module:ESP32-S2-WROVER, symbol Device:R_US
- added R35: 10k, RF_Module:ESP32-S2-WROVER, symbol Device:R_US
Connections:
- net GND: now also Q24.3 (S), R35.1
- new net: Q24.2 (G), R34.2, R35.2
- new net +3.3V: Q24.1 (D)
- new net electromagnet: R34.1

Commit message: add
Parts:
- renumbered J6 to J10, J7 to J11, J9 to J12, J15 to J13, J12 to J14, J8 to J3, J5 to J4, J4 to J5, J10 to J6, J14 to J7, J3 to J8, J11 to J9, Q16 to Q10, Q10 to Q11, Q17 to Q12, Q11 to Q13, Q12 to Q14, Q24 to Q15, Q13 to Q16, Q14 to Q17, Q15 to Q8, R28 to R30, R29 to R31, R38 to R32, R22 to R33, R30 to R34, R31 to R35, R39 to R36, R23 to R37, R40 to R38, R32 to R39, R24 to R40, R33 to R41, R41 to R42, R25 to R43, R34 to R44, R35 to R45, R26 to R46, R27 to R47

Commit message: Almost done with Schematic
Parts:
- removed Q10, Q12, Q15, Q8: NMOS, Package_DFN_QFN:SiliconLabs_QFN-20-1EP_3x3mm_P0.5mm, symbol Simulation_SPICE:NMOS
- added J15: Conn_01x02_Pin, symbol Connector:Conn_01x02_Pin
- added Q18, Q19, Q20, Q21: BSS138, Package_TO_SOT_SMD:SOT-23, symbol Transistor_FET:BSS138
- J10, J11, J12, J14, J4, J5, J8: footprint Package_DFN_QFN:QFN-20-1EP_5x5mm_P0.65mm_EP3.35x3.35mm -> (none)
- J13, J7: footprint Connector:Tag-Connect_TC2030-IDC-FP_2x03_P1.27mm_Vertical -> (none)
- J6, J9: footprint Converter_DCDC:Converter_DCDC_Cyntec_MUN12AD01-SH -> (none)
- R30, R31, R32, R34, R35, R36, R38, R39, R41, R42, R44, R45: footprint RF_Module:ESP32-S2-WROVER -> Resistor_SMD:R_0603_1608Metric_Pad0.98x0.95mm_HandSolder
- R33, R37, R40, R43, R46, R47: footprint Package_TO_SOT_SMD:SOT-23 -> Resistor_SMD:R_0603_1608Metric_Pad0.98x0.95mm_HandSolder
Connections:
- net +24V: now also J15.2 (Pin_2)
- net GND: now also Q18.2 (S), Q19.2 (S), Q20.2 (S), Q21.2 (S)
- net at R34.2, R35.2: now also Q19.1 (G)
- net at J3.1 (Pin_1): now also Q18.3 (D)
- net at R30.2, R31.2: now also Q18.1 (G)
- net at J6.1 (Pin_1): now also Q19.3 (D)
- net at J9.1 (Pin_1): now also Q20.3 (D)
- net at R39.2, R41.2: now also Q20.1 (G)
- net at R44.2, R45.2: now also Q21.1 (G)
- new net: J15.1 (Pin_1), Q21.3 (D)
Other:
- moved on the sheet: J12

Commit message: add
Parts:
- J10, J13, J4, J5, J7, J8: footprint (none) -> Connector_JST:JST_PH_B4B-PH-K_1x04_P2.00mm_Vertical
- J11, J12, J14, J15, J6, J9: footprint (none) -> Connector_JST:JST_PH_B2B-PH-K_1x02_P2.00mm_Vertical
Changed lines of the file:
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@@
 			)
 		)
-		(property "Footprint" ""
+		(property "Footprint" "Connector_JST:JST_PH_B2B-PH-K_1x02_P2.00mm_Vertical"
 			(at 259.08 41.91 0)
 			(hide yes)
@@
 			)
 		)
-		(property "Footprint" ""
+		(property "Footprint" "Connector_JST:JST_PH_B2B-PH-K_1x02_P2.00mm_Vertical"
 			(at 102.87 95.25 0)
 			(hide yes)
@@
 			)
 		)
-		(property "Footprint" ""
+		(property "Footprint" "Connector_JST:JST_PH_B4B-PH-K_1x04_P2.00mm_Vertical"
 			(at 57.15 52.07 0)
 			(hide yes)
@@
 			)
 		)
-		(property "Footprint" ""
+		(property "Footprint" "Connector_JST:JST_PH_B4B-PH-K_1x04_P2.00mm_Vertical"
 			(at 95.25 52.07 0)
 			(hide yes)
@@
 			)
 		)
-		(property "Footprint" ""
+		(property "Footprint" "Connector_JST:JST_PH_B2B-PH-K_1x02_P2.00mm_Vertical"
 			(at 213.36 41.91 0)
 			(hide yes)
@@
 			)
 		)
-		(property "Footprint" ""
+		(property "Footprint" "Connector_JST:JST_PH_B2B-PH-K_1x02_P2.00mm_Vertical"
 			(at 152.4 95.25 0)
 			(hide yes)
@@
 			)
 		)
-		(property "Footprint" ""
+		(property "Footprint" "Connector_JST:JST_PH_B2B-PH-K_1x02_P2.00mm_Vertical"
 			(at 255.27 80.01 0)
 			(hide yes)
@@
 			)
 		)
-		(property "Footprint" ""
+		(property "Footprint" "Connector_JST:JST_PH_B4B-PH-K_1x04_P2.00mm_Vertical"
 			(at 173.99 52.07 0)
 			(hide yes)
@@
 			)
 		)
-		(property "Footprint" ""
+		(property "Footprint" "Connector_JST:JST_PH_B4B-PH-K_1x04_P2.00mm_Vertical"
 			(at 133.35 52.07 0)
 			(hide yes)
@@
 			)
 		)
-		(property "Footprint" ""
+		(property "Footprint" "Connector_JST:JST_PH_B4B-PH-K_1x04_P2.00mm_Vertical"
 			(at 250.19 116.84 0)
 			(hide yes)
@@
 			)
 		)
-		(property "Footprint" ""
+		(property "Footprint" "Connector_JST:JST_PH_B4B-PH-K_1x04_P2.00mm_Vertical"
 			(at 121.92 153.67 0)
 			(hide yes)
@@
 			)
 		)
-		(property "Footprint" ""
+		(property "Footprint" "Connector_JST:JST_PH_B2B-PH-K_1x02_P2.00mm_Vertical"
 			(at 210.82 81.28 0)
 			(hide yes)
