File: core_board/Power_in.kicad_sch (KiCad schematic)
At the start: 1 part, among them J1 Molex_Megafit_02

Commit message: Finish Power Schematic
Parts:
- added C1, C7: 10uF, Package_SO:SOIC-8_3.9x4.9mm_P1.27mm, symbol Device:C
- added C2, C4: 100nF, Package_SO:SOIC-8_3.9x4.9mm_P1.27mm, symbol Device:C
- added C3, C6, C8, C9: 22uF, Package_SO:SOIC-8_3.9x4.9mm_P1.27mm, symbol Device:C
- added C5: 47pF, Package_SO:SOIC-8_3.9x4.9mm_P1.27mm, symbol Device:C
- added D1: MMSZ5240BT1G, MRDT_Devices:SOD-123_ONS-L, symbol MRDT_Devices:MMSZ5240BT1G
- added GreenLED1: LED, symbol Device:LED
- added GreenLED2, GreenLED3: LED, LED_SMD:LED_Cree-XHP50_3V_HighDensity, symbol Device:LED
- added L1: 4.7uH, OptoDevice:Everlight_ITR9608-F, symbol Device:L
- added L2: 10uH, OptoDevice:Everlight_ITR9608-F, symbol Device:L
- added Q1: TPC8132_LQS, MRDT_Devices:TPC8132_LQS, symbol MRDT_Devices:TPC8132_LQS
- added R1: 6.8K, Package_DIP:DIP-8_W7.62mm, symbol Device:R_US
- added R2: 2.2K, Package_DIP:DIP-8_W7.62mm, symbol Device:R_US
- added R3: 1.5K, Package_DIP:DIP-8_W7.62mm, symbol Device:R_US
- added R4: 1k, Package_DIP:DIP-8_W7.62mm, symbol Device:R_US
- added R5: 252K, Package_DIP:DIP-8_W7.62mm, symbol Device:R_US
- added R6: 30.1k, Package_DIP:DIP-8_W7.62mm, symbol Device:R_US
- added U1: AP63205QWU7, AP63205QWU7:SOT95P280X100-6N, symbol AP63205QWU7:AP63205QWU7
- added U2: AP63301WU7, AP63205QWU7:SOT95P280X100-6N, symbol AP63205QWU7:AP63205QWU7
Connections:
- net +24V: now also C1.1, C7.1, D1.1, Q1.S, R1.1, U1.2 (EN), U1.3 (VIN), U2.2 (EN), U2.3 (VIN); no longer J1.2
- net GND: now reaches J1.1
- net GND: now also C1.2, C3.2, C6.2, C7.2, C8.2, C9.2, GreenLED1.1 (K), GreenLED2.1 (K), GreenLED3.1 (K), R4.2, R6.2, U1.4 (GND), U2.4 (GND)
- new net: GreenLED2.2 (A), R2.2
- new net: D1.2, Q1.G, R4.1
- new net: C5.2, R5.2, R6.1, U2.1 (FB)
- new net: GreenLED1.2 (A), R1.2
- new net: C2.1, L1.1, U1.5 (SW)
- new net: C2.2, U1.6 (BST)
- new net: C4.1, L2.1, U2.5 (SW)
- new net: C4.2, U2.6 (BST)
- new net: GreenLED3.2 (A), R3.2
- new net: J1.2, Q1.D
- new net +5V: C3.1, C9.1, L1.2, R3.1, U1.1 (FB)
- new net +7.5V: C5.1, C6.1, C8.1, L2.2, R2.1, R5.1
Changed lines of the file:
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@@
 	(generator_version "10.0")
 	(paper "A4")
-	(wire
-		(pts
-			(xy 39.37 43.18) (xy 45.72 43.18)
-		)
-		(stroke
-			(width 0)
-			(type default)
-		)
-	)
-	(wire
-		(pts
-			(xy 45.72 43.18) (xy 45.72 39.37)
-		)
-		(stroke
-			(width 0)
-			(type default)
-		)
-	)
-	(symbol
-		(lib_id "power:+24V")
-		(at 45.72 39.37 0)
-		(unit 1)
-		(body_style 1)
-		(exclude_from_sim no)
-		(in_bom yes)
-		(on_board yes)
-		(in_pos_files yes)
-		(dnp no)
-		(fields_autoplaced yes)
-		(property "Reference" "#PWR01"
-			(at 45.72 43.18 0)
-			(hide yes)
-			(show_name no)
-			(do_not_autoplace no)
-			(effects
-				(font
-					(size 1.27 1.27)
-				)
-			)
-		)
-		(property "Value" "+24V"
-			(at 45.72 34.29 0)
-			(show_name no)
-			(do_not_autoplace no)
-			(effects
-				(font
-					(size 1.27 1.27)
-				)
-			)
-		)
-		(property "Footprint" ""
-			(at 45.72 39.37 0)
-			(hide yes)
-			(show_name no)
-			(do_not_autoplace no)
-			(effects
-				(font
-					(size 1.27 1.27)
-				)
-			)
-		)
-		(property "Datasheet" ""
-			(at 45.72 39.37 0)
-			(hide yes)
-			(show_name no)
-			(do_not_autoplace no)
-			(effects
-				(font
-					(size 1.27 1.27)
-				)
-			)
-		)
-		(property "Description" "Power symbol creates a global label with name \"+24V\""
-			(at 45.72 39.37 0)
-			(hide yes)
-			(show_name no)
-			(do_not_autoplace no)
-			(effects
-				(font
-					(size 1.27 1.27)
-				)
-			)
-		)
-		(pin "1"
-		)
-		(instances
-			(project "core_board"
-				(path "/e01d6047-065c-44c8-9643-8ab57e6ffae6/99860962-d8ec-450a-a69d-1c445546f8f2"
-					(reference "#PWR01")
-					(unit 1)
-				)
-			)
-		)
-	)
-	(symbol
-		(lib_id "MRDT_Connectors:Molex_Megafit_02")
-		(at 39.37 45.72 180)
-		(unit 1)
-		(body_style 1)
-		(exclude_from_sim no)
-		(in_bom yes)
-		(on_board yes)
-		(in_pos_files yes)
-		(dnp no)
-		(fields_autoplaced yes)
-		(property "Reference" "J1"
-			(at 30.48 35.56 0)
-			(show_name no)
-			(do_not_autoplace no)
-			(effects
-				(font
-					(size 1.524 1.524)
-				)
-			)
-		)
-		(property "Value" "Molex_Megafit_02"
-			(at 30.48 38.1 0)
-			(show_name no)
-			(do_not_autoplace no)
-			(effects
-				(font
-					(size 1.524 1.524)
-				)
-			)
-		)
-		(property "Footprint" "MRDT_Connectors:MOLEX_MegaFit_02_Horizontal"
-			(at 39.37 45.72 0)
-			(hide yes)
-			(show_name no)
-			(do_not_autoplace no)
-			(effects
-				(font
-					(size 1.27 1.27)
-					(italic yes)
-				)
-			)
-		)
-		(property "Datasheet" "https://www.molex.com/en-us/products/part-detail-pdf/768250002?display=pdf"
-			(at 39.37 45.72 0)
-			(hide yes)
-			(show_name no)
-			(do_not_autoplace no)
-			(effects
-				(font
-					(size 1.27 1.27)
-					(italic yes)
-				)
-			)
-		)
-		(property "Description" ""
-			(at 39.37 45.72 0)
-			(hide yes)
-			(show_name no)
-			(do_not_autoplace no)
-			(effects
-				(font
-					(size 1.27 1.27)
-				)
-			)
-		)
-		(pin "1"
-		)
-		(pin "2"
-		)
-		(instances
-			(project "core_board"
-				(path "/e01d6047-065c-44c8-9643-8ab57e6ffae6/99860962-d8ec-450a-a69d-1c445546f8f2"
-					(reference "J1")
-					(unit 1)
-				)
-			)
-		)
-	)
-)

Commit message: Finish Ethernet, Servo Motors, CAN Connector, and SMOCO
Started fans but still need to finalize what type of fan we are using. Microcontroller started still need finished.
Other:
- note added: "BUCK CONVERTERS"
- note added: "LEDS"
- note added: "REVERSE VOLTAGE PROTECTION"
- moved on the sheet: C3, C6, GreenLED1, GreenLED2, GreenLED3, R1, R2, R3

Commit message: finish stuff
Parts:
- L2: value 10uH -> 14uH

Commit message: add
Parts:
- renumbered C7 to C1, C1 to C2, C4 to C3, C2 to C4, C3 to C6, C9 to C7, C6 to C8, C8 to C9, L2 to L1, L1 to L2, R4 to R1, R5 to R2, R6 to R3, R1 to R4, R2 to R5, R3 to R6, U2 to U1, U1 to U2

Commit message: New buck I think
Trying to make buck work
Parts:
- added C12, C13, C14, C15: C_Small, Package_SO:SOIC-8_3.9x4.9mm_P1.27mm, symbol Device:C_Small
- added D12: MMSZ5240BT1G, MRDT_Devices:SOD-123_ONS-L, symbol MRDT_Devices:MMSZ5240BT1G
- added L3: 4.7uH, OptoDevice:Everlight_ITR9608-F, symbol Device:L
- added R48, R50, R51, R52: R_US, Package_DFN_QFN:WDFN-10-1EP_3x3mm_P0.5mm_EP1.8x2.5mm, symbol Device:R_US
- added R49: R_US, symbol Device:R_US
- added U4: AOZ6605PI-1, SOIC-8:SO8_EP1_AOS, symbol 8-SOIC:AOZ6605PI-1
- GreenLED1: footprint (none) -> Inductor_SMD:L_0603_1608Metric_Pad1.05x0.95mm_HandSolder
- GreenLED2, GreenLED3: footprint LED_SMD:LED_Cree-XHP50_3V_HighDensity -> LED_SMD:LED_0603_1608Metric_Pad1.05x0.95mm_HandSolder
Connections:
- net +24V: now also C15.1, R51.1, U4.6 (VCC)
- net +5V: now also C13.1, L3.2, R48.1
- net GND: now also C13.2, C15.2, D12.2, R49.2, R50.2, R52.2, U4.4 (GND)
- new net: C14.1, U4.5 (BST)
- new net: C14.2, D12.1, L3.1, U4.EPAD (LX)
- new net: C12.2, R50.1
- new net: R48.2, R49.1, U4.8 (FB)
- new net: R51.2, R52.1, U4.2 (EN)
- new net: C12.1, U4.3 (VC)

Commit message: Almost done with Schematic
Parts:
- removed R51, R52: R_US, Package_DFN_QFN:WDFN-10-1EP_3x3mm_P0.5mm_EP1.8x2.5mm, symbol Device:R_US
- C1, C12, C13, C14, C15, C2, C3, C4, C5, C6, C7, C8, C9: footprint Package_SO:SOIC-8_3.9x4.9mm_P1.27mm -> Capacitor_SMD:C_0603_1608Metric_Pad1.08x0.95mm_HandSolder
- D1, D12: footprint MRDT_Devices:SOD-123_ONS-L -> LED_SMD:LED_0603_1608Metric_Pad1.05x0.95mm_HandSolder
- GreenLED1: footprint Inductor_SMD:L_0603_1608Metric_Pad1.05x0.95mm_HandSolder -> LED_SMD:LED_0603_1608Metric_Pad1.05x0.95mm_HandSolder
- L1, L2: footprint OptoDevice:Everlight_ITR9608-F -> (none)
- L3: value 4.7uH -> 22uH; footprint OptoDevice:Everlight_ITR9608-F -> AMRM00101040220MA1:IND_AMRM00101040_PUL
- R1, R2, R3, R4, R5, R6: footprint Package_DIP:DIP-8_W7.62mm -> Resistor_SMD:R_0603_1608Metric_Pad0.98x0.95mm_HandSolder
- R48, R50: footprint Package_DFN_QFN:WDFN-10-1EP_3x3mm_P0.5mm_EP1.8x2.5mm -> Resistor_SMD:R_0603_1608Metric_Pad0.98x0.95mm_HandSolder
- R49: footprint (none) -> Resistor_SMD:R_0603_1608Metric_Pad0.98x0.95mm_HandSolder
- U1, U2: footprint AP63205QWU7:SOT95P280X100-6N -> Package_TO_SOT_SMD:SOT-23-6_Handsoldering
- U4: value AOZ6605PI-1 -> BD9G401EFJ-E2; footprint SOIC-8:SO8_EP1_AOS -> Package_SO:SOIC-8-1EP_3.9x4.9mm_P1.27mm_EP2.29x3mm
Connections:
- net +24V: now also U4.8 (VCC); no longer U4.6 (VCC)
- net GND: now also U4.2 (GND), U4.5 (SYNC), U4.EPAD (THML_PAD); no longer U4.4 (GND)
- net at C14.1: now also U4.7 (BST); no longer U4.5 (BST)
- net at C14.2, D12.1, L3.1: now also U4.1 (LX); no longer U4.EPAD (LX)
- net at R48.2, R49.1: now also U4.4 (FB); no longer U4.8 (FB)
- new net +3V3: U4.6 (EN)
Other:
- moved on the sheet: C12, C13, C14, C15, C2, C4, C6, C7, D12, L2, L3, R48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

Commit message: add
Parts:
- L1: footprint (none) -> Inductor_SMD:L_TechFuse_SL1050
- L2: footprint (none) -> Inductor_SMD:L_0603_1608Metric
