File: core_board/Microcontroller.kicad_sch (KiCad schematic)
At the start: 3 parts, among them J2 RJ45_LED_Shielded

Commit message: Finish Schematic
Connections:
- net Fan1PWM: now also U4.29 (PB7); no longer U4.30 (PB8)
- net Fan2PWM: now also U4.28 (PB6); no longer U4.29 (PB7)
- net Fan3PWM: now also U4.27 (PB5); no longer U4.28 (PB6)
- net RED_PWM_StateDisplay: now reaches U4.13 (PC9)
- net BLUE_PWM_StateDisplay: now reaches U4.14 (PC8)
- net LeftPAN_PWM: now reaches U4.16 (PC6)
- net Spare1_PWM: now reaches U4.17 (PB14)
- net SMOCO_LED: now reaches U4.18 (PB13)
- net RTRY4: now reaches U4.25 (PD2)
- net RTRY2: now reaches U4.26 (PB4)
- net PanLeft_LED: now reaches U4.35 (PH1)
- net TiltBack_LED: now reaches U4.36 (PC2)
- net TiltRight_LED: now reaches U4.37 (PC3)
- net CANLow: now reaches U4.4 (CAN_L)
- net LeftTilt_PWM: now reaches U4.42 (PB0)
- net RightPAN_PWM: now reaches U4.43 (PB1)
- net PanBack_LED: now reaches U4.44 (PB2)
- net CANHigh: now reaches U4.5 (CAN_H)
- net Direction_Switch: now reaches U4.6 (PC12)
- net Up: now reaches U4.7 (PC11)
- net Down: now reaches U4.8 (PC10)
- net BackPan_PWM: now reaches U4.9 (PA15)
- net BackPan renamed BackTilt_PWM
- net BackTilt renamed GREEN_PWM_StateDisplay
- net Ledout1 renamed Left
- net Ledout2 renamed Right
- net Ledout3 renamed PanRight_LED
- net Ledout4 renamed TEMP_OUT
- net LeftPAN renamed RED_PWM_Internal
- net LeftTilt renamed GREEN_PWM_Internal
- net RightPAN renamed BLUE_PWM_Internal
- net RightTilt renamed TiltLeft_LED
- net Spare1 renamed Spare2_PWM
- net Spare2 renamed RightTilt_PWM
- new net RTRY1: U4.30 (PB8)
- no-connect marks 1 -> 2

Commit message: Change TEMP_OUT from Pin PH0 to PA4
Connections:
- net TEMP_OUT: now also U4.40 (PA4); no longer U4.34 (PH0)
Changed lines of the file:
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@@
 	)
 	(no_connect
-		(at 92.71 80.01)
+		(at 92.71 63.5)
 	)
 	(wire
@@
 	(wire
 		(pts
-			(xy 88.9 63.5) (xy 92.71 63.5)
-		)
-		(stroke
-			(width 0)
-			(type default)
-		)
-	)
-	(wire
-		(pts
 			(xy 120.65 64.77) (xy 116.84 64.77)
 		)
@@
 		(pts
 			(xy 209.55 58.42) (xy 209.55 62.23)
+		)
+		(stroke
+			(width 0)
+			(type default)
+		)
+	)
+	(wire
+		(pts
+			(xy 88.9 80.01) (xy 92.71 80.01)
 		)
 		(stroke
@@
 	(hierarchical_label "TEMP_OUT"
 		(shape input)
-		(at 88.9 63.5 180)
-		(effects
-			(font
+		(at 88.9 80.01 180)
+		(effects
+			(font

Commit message: add
Connections:
- net Spare1_PWM renamed electromagnet
Changed lines of the file:
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@@
+		)
+	)
+	(hierarchical_label "electromagnet"
+		(shape output)
+		(at 120.65 82.55 0)
+		(effects
+			(font
+				(size 1.27 1.27)
+			)
+			(justify left)
 		)
 	)
@@
 		)
 	)
-	(hierarchical_label "Spare1_PWM"
-		(shape output)
-		(at 120.65 82.55 0)
-		(effects
-			(font
-				(size 1.27 1.27)
-			)
-			(justify left)
-		)
-	)

Commit message: add
Parts:
- renumbered C10 to C11, U4 to U3
Changed lines of the file:
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@@
 		(dnp no)
 		(fields_autoplaced yes)
-		(property "Reference" "U4"
+		(property "Reference" "U3"
 			(at 104.775 31.75 0)
 			(show_name no)
@@
 			(project "core_board"
 				(path "/e01d6047-065c-44c8-9643-8ab57e6ffae6/484197b8-3571-44f1-846b-0b6f9c5f5a1e"
-					(reference "U4")
+					(reference "U3")
 					(unit 1)
 				)
@@
 		(dnp no)
 		(fields_autoplaced yes)
-		(property "Reference" "C10"
+		(property "Reference" "C11"
 			(at 215.9 73.6599 0)
 			(show_name no)
@@
 			(project "core_board"
 				(path "/e01d6047-065c-44c8-9643-8ab57e6ffae6/484197b8-3571-44f1-846b-0b6f9c5f5a1e"
-					(reference "C10")
+					(reference "C11")
 					(unit 1)
 				)
@@
 		(dnp no)
 		(fields_autoplaced yes)
-		(property "Reference" "#PWR022"
+		(property "Reference" "#PWR051"
 			(at 127 38.1 0)
 			(hide yes)
@@
 			(project "core_board"
 				(path "/e01d6047-065c-44c8-9643-8ab57e6ffae6/484197b8-3571-44f1-846b-0b6f9c5f5a1e"
-					(reference "#PWR022")
+					(reference "#PWR051")
 					(unit 1)
 				)
@@
 		(dnp no)
 		(fields_autoplaced yes)
-		(property "Reference" "#PWR021"
+		(property "Reference" "#PWR052"
 			(at 133.35 49.53 0)
 			(hide yes)
@@
 			(project "core_board"
 				(path "/e01d6047-065c-44c8-9643-8ab57e6ffae6/484197b8-3571-44f1-846b-0b6f9c5f5a1e"
-					(reference "#PWR021")
+					(reference "#PWR052")
 					(unit 1)
 				)
@@
 		(dnp no)
 		(fields_autoplaced yes)
-		(property "Reference" "#PWR020"
+		(property "Reference" "#PWR050"
 			(at 121.92 38.1 0)
 			(hide yes)
@@
 			(project "core_board"
 				(path "/e01d6047-065c-44c8-9643-8ab57e6ffae6/484197b8-3571-44f1-846b-0b6f9c5f5a1e"
-					(reference "#PWR020")
+					(reference "#PWR050")
 					(unit 1)
 				)
@@
 		(dnp no)
 		(fields_autoplaced yes)
-		(property "Reference" "#PWR023"
+		(property "Reference" "#PWR053"
 			(at 212.09 91.44 0)
 			(hide yes)
@@
 			(project "core_board"
 				(path "/e01d6047-065c-44c8-9643-8ab57e6ffae6/484197b8-3571-44f1-846b-0b6f9c5f5a1e"
-					(reference "#PWR023")
+					(reference "#PWR053")
 					(unit 1)
 				)

Commit message: Add extra components
fixed LED connector
removed extra buck
fixed wrong footprints
Parts:
- J2: footprint Connector_RJ:RJ45_Abracon_ARJP11A-MA_Horizontal -> MRDT_Connectors:RJ45_Teensy
Connections:
- net BLUE_PWM_Internal: no longer names the net of U3.10 (PA10)
- net BLUE_PWM_StateDisplay renamed InternalLighting_PWM
- net GREEN_PWM_Internal: no longer names the net of U3.11 (PA9)
- net GREEN_PWM_StateDisplay renamed StateDisplay_PWM
- net RED_PWM_Internal: no longer names the net of U3.12 (PA8)
- net RED_PWM_StateDisplay renamed SparePWM1
Changed lines of the file:
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@@
-	(wire
-		(pts
-			(xy 120.65 67.31) (xy 116.84 67.31)
-		)
-		(stroke
-			(width 0)
-			(type default)
-		)
-	)
 	(wire
 		(pts
@@
 	(wire
 		(pts
-			(xy 120.65 64.77) (xy 116.84 64.77)
-		)
-		(stroke
-			(width 0)
-			(type default)
-		)
-	)
-	(wire
-		(pts
 			(xy 88.9 44.45) (xy 92.71 44.45)
 		)
@@
 		(pts
 			(xy 116.84 91.44) (xy 119.38 91.44)
-		)
-		(stroke
-			(width 0)
-			(type default)
-		)
-	)
-	(wire
-		(pts
-			(xy 120.65 69.85) (xy 116.84 69.85)
 		)
 		(stroke
@@
 		)
 	)
-	(hierarchical_label "RED_PWM_Internal"
-		(shape output)
-		(at 120.65 69.85 0)
-		(effects
-			(font
-				(size 1.27 1.27)
-			)
-			(justify left)
-		)
-	)
 	(hierarchical_label "TEMP_OUT"
 		(shape input)
@@
 		)
 	)
-	(hierarchical_label "BLUE_PWM_Internal"
-		(shape output)
-		(at 120.65 64.77 0)
-		(effects
-			(font
-				(size 1.27 1.27)
-			)
-			(justify left)
-		)
-	)
 	(hierarchical_label "LeftPAN_PWM"
 		(shape output)
@@
 		)
 	)
-	(hierarchical_label "GREEN_PWM_StateDisplay"
+	(hierarchical_label "StateDisplay_PWM"
 		(shape output)
 		(at 120.65 77.47 0)
@@
 		)
 	)
-	(hierarchical_label "RED_PWM_StateDisplay"
+	(hierarchical_label "SparePWM1"
 		(shape output)
 		(at 120.65 72.39 0)
@@
 		)
 	)
-	(hierarchical_label "BLUE_PWM_StateDisplay"
+	(hierarchical_label "InternalLighting_PWM"
 		(shape output)
 		(at 120.65 74.93 0)
@@
 			)
 			(justify right)
-		)
-	)
-	(hierarchical_label "GREEN_PWM_Internal"
-		(shape output)
-		(at 120.65 67.31 0)
-		(effects
-			(font
-				(size 1.27 1.27)
-			)
-			(justify left)
 		)
 	)
@@
 			)
 		)
-		(property "Footprint" "Connector_RJ:RJ45_Abracon_ARJP11A-MA_Horizontal"
+		(property "Footprint" "MRDT_Connectors:RJ45_Teensy"
 			(at 217.805 48.26 90)
 			(hide yes)
