File: core_board/core_board.kicad_pcb (KiCad board)
At the start: 2 copper layers, 111 parts, among them J1 Molex_Megafit_02, J10 Conn_01x04_Pin, J11 Conn_01x02_Pin, J12 Conn_01x02_Pin, J13 Conn_01x03_Pin, J14 Conn_01x02_Pin, J15 Conn_01x02_Pin, J16 Conn_01x03_Pin, J2 RJ45_LED_Shielded, J3 Conn_01x02_Pin, J4Serv1 Conn_01x04_Pin, J5 Conn_01x04_Pin, J6 Conn_01x02_Pin, J8 Conn_01x04_Pin, J9 Conn_01x02_Pin, Q1 TPC8132_LQS, Q18 BSS138, Q19 BSS138, Q2 BSS138, Q20 BSS138, Q21 BSS138, Q3 BSS138, Q4 BSS138, Q5 BSS138, Q6 BSS138, Q7 BSS138, SW1 SW_Push, SW2 SW_Push, SW3 SW_Push, SW4 SW_Push, U1 AP63301WU7, U4 BD9G401EFJ-E2

Commit message: add
Parts:
- moved U5 4.29 mm to (197.6, 25.9)
- moved U7 4.02 mm to (86.8, 141.8)
- moved U6 2.46 mm to (197.5, 141.9)
- moved U8 0.85 mm to (86.9, 25.9)
Other:
- board outline added: 221 x 177.8 mm
Changed lines of the file:
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@@
 	(footprint "MRDT_Drill_Holes:4_40_Hole_Pad_Via"
 		(layer "F.Cu")
-		(at 195.497056 29.647056)
+		(at 197.595713 25.89991)
 		(property "Reference" "U5"
 			(at 0 -0.5 0)
@@
 	(footprint "MRDT_Drill_Holes:4_40_Hole_Pad_Via"
 		(layer "F.Cu")
-		(at 197.697056 144.352944)
+		(at 197.489744 141.905056)
 		(property "Reference" "U6"
 			(at 0 -0.5 0)
@@
 	(footprint "MRDT_Drill_Holes:4_40_Hole_Pad_Via"
 		(layer "F.Cu")
-		(at 90.85 141.8)
+		(at 86.82671 141.797539)
 		(property "Reference" "U7"
 			(at 0 -0.5 0)
@@
 	(footprint "MRDT_Drill_Holes:4_40_Hole_Pad_Via"
 		(layer "F.Cu")
-		(at 87.3 26.6)
+		(at 86.85991 25.873487)
 		(property "Reference" "U8"
 			(at 0 -0.5 0)
@@
 		)
 	)
+	(gr_line
+		(start 81.28 142.24038)
+		(end 81.286375 25.818302)
+		(stroke
+			(width 0.05)
+			(type solid)
+		)
+		(layer "Edge.Cuts")
+	)
+	(gr_arc
+		(start 81.286375 25.818302)
+		(mid 82.772662 22.083798)
+		(end 86.384392 20.32)
+		(stroke
+			(width 0.05)
+			(type default)
+		)
+		(layer "Edge.Cuts")
+	)
+	(gr_line
+		(start 86.384392 20.32)
+		(end 198.0184 20.32)
+		(stroke
+			(width 0.05)
+			(type solid)
+		)
+		(layer "Edge.Cuts")
+	)
+	(gr_arc
+		(start 86.77162 147.361581)
+		(mid 82.8548 145.6944)
+		(end 81.262629 141.746494)
+		(stroke
+			(width 0.05)
+			(type solid)
+		)
+		(layer "Edge.Cuts")
+	)
+	(gr_arc
+		(start 197.650896 20.326375)
+		(mid 201.5744 21.9964)
+		(end 203.169287 25.951044)
+		(stroke
+			(width 0.05)
+			(type default)
+		)
+		(layer "Edge.Cuts")
+	)
+	(gr_line
+		(start 198.095349 147.32)
+		(end 86.77162 147.361581)
+		(stroke
+			(width 0.05)
+			(type solid)
+		)
+		(layer "Edge.Cuts")
+	)
+	(gr_arc
+		(start 203.193625 141.821696)
+		(mid 201.5236 145.7452)
+		(end 197.568956 147.340087)
+		(stroke
+			(width 0.05)
+			(type default)
+		)
+		(layer "Edge.Cuts")
+	)
+	(gr_line
+		(start 203.2 25.4)
+		(end 203.193625 141.821696)
+		(stroke
+			(width 0.05)
+			(type default)
+		)
+		(layer "Edge.Cuts")
+	)
+	(gr_line
+		(start 203.2 25.5016)
+		(end 203.2 25.4)
+		(stroke
+			(width 0.05)
+			(type default)
+		)
+		(layer "Edge.Cuts")
+	)
+	(gr_line
+		(start 302.26 -30.48)
+		(end 302.26 -27.94)
+		(stroke
+			(width 0.05)
+			(type default)
+		)
+		(layer "Edge.Cuts")
+	)
 	(gr_text "PCB Editor"
 		(at 154.05 169.1 0)
@@
 		(layer "B.Paste")
 	)
+	(point
+		(at 83.82 5.08)
+		(size 1)
+		(layer "Edge.Cuts")
+	)
 	(embedded_fonts no)

Commit message: add
Routing:
- added copper zone on B.Cu, net GND
- added copper zone on F.Cu, net GND
Changed lines of the file:
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@@
 		(layer "Edge.Cuts")
+	)
+	(zone
+		(net "GND")
+		(layers "F.Cu" "B.Cu")
+		(hatch edge 0.5)
+		(connect_pads yes
+			(clearance 0.254)
+		)
+		(min_thickness 0.1778)
+		(fill yes
+			(thermal_gap 0.5)
+			(thermal_bridge_width 0.5)
+			(island_removal_mode 0)
+		)
+		(polygon
+			(pts
+				(xy 81.28 19.6088) (xy 83.9724 19.6088) (xy 203.655741 20.344343) (xy 202.407056 147.004386) (xy 202.407053 147.004387)
+				(xy 80.580151 147.229106) (xy 80.564109 147.213972) (xy 80.4672 20.1168) (xy 80.4672 19.6088)
+			)
+		)
 	)
 	(embedded_fonts no)
