File: core_board/testing buttons.kicad_sch (KiCad schematic)
At the start: 45 parts, among them Q19 NMOS, Q2 PMOS, Q3 PMOS, Q4 PMOS, Q5 PMOS, Q6 PMOS, Q7 PMOS, Q8 PMOS, SW1 SW_Push, SW2 SW_Push, SW3 SW_Push, SW4 SW_Push

Commit message: add
Parts:
- removed D10, D11, D12, D6, D7, D8, D9: Blue, symbol Device:LED
- removed Q19: NMOS, symbol Simulation_SPICE:NMOS
- removed Q2, Q3, Q4, Q5, Q6, Q7, Q8: PMOS, symbol Simulation_SPICE:PMOS
- removed R11, R12, R13, R14, R15, R17, R21: 1k, symbol Device:R_US
- removed R18, R19, R20, R34, R35, R36, R37: 10k, symbol Device:R_US
- added D14, D15, D16, D17, D18: Blue, symbol Device:LED
- added Q18, Q19, Q20, Q21, Q22, Q23: BSS138, Package_TO_SOT_SMD:SOT-23, symbol Transistor_FET:BSS138
- added R40, R42, R45, R48, R51, R54: 100, symbol Device:R_US
- added R41, R44, R47, R50, R53: 10k, symbol Device:R_US
- added R43, R46, R49, R52, R55: 1k, symbol Device:R_US
Connections:
- net +3V3: now also D13.2 (A), D14.2 (A), D15.2 (A), D16.2 (A), D17.2 (A), D18.2 (A); no longer D13.1 (K)
- net GND: now also R38.2, Q18.2 (S), Q19.2 (S), Q20.2 (S), Q21.2 (S), Q22.2 (S), Q23.2 (S), R41.2, R44.2, R47.2, R50.2, R53.2
- net PanBack_LED: now also R41.1, R42.1
- net PanLeft_LED: now also R44.1, R45.1
- net SMOCO_LED: now also R38.1, R40.1
- net TiltBack_LED: now also R50.1, R51.1
- net TiltLeft_LED: now also R47.1, R48.1
- net TiltRight_LED: now also R53.1, R54.1
- net at R39.1: now also D13.1 (K); no longer D13.2 (A)
- net at R39.2: now also Q18.3 (D)
- new net: D14.1 (K), R43.1
- new net: D15.1 (K), R46.1
- new net: Q19.3 (D), R43.2
- new net: Q19.1 (G), R42.2
- new net: Q22.1 (G), R51.2
- new net: Q22.3 (D), R52.2
- new net: Q20.3 (D), R46.2
- new net: Q23.1 (G), R54.2
- new net: D17.1 (K), R52.1
- new net: D16.1 (K), R49.1
- new net: Q21.3 (D), R49.2
- new net: Q18.1 (G), R40.2
- new net: Q20.1 (G), R45.2
- new net: Q21.1 (G), R48.2
- new net: D18.1 (K), R55.1
- new net: Q23.3 (D), R55.2
- no-connect marks 3 -> 1

Commit message: add
Connections:
- no-connect marks 1 -> 2
Changed lines of the file:
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@@
 		(at 57.15 134.62)
+	)
+	(no_connect
+		(at 144.78 125.73)
 	)
 	(wire

Commit message: add
Parts:
- renumbered D15 to D10, D17 to D11, D4 to D3, D3 to D4, D13 to D6, D14 to D7, D16 to D8, D18 to D9, Q18 to Q2, Q19 to Q3, Q21 to Q4, Q23 to Q5, Q20 to Q6, Q22 to Q7, R8 to R10, R38 to R11, R9 to R12, R40 to R13, R39 to R14, R41 to R15, R47 to R16, R42 to R17, R48 to R18, R43 to R19, R49 to R20, R53 to R21, R54 to R22, R44 to R23, R45 to R24, R55 to R25, R46 to R26, R50 to R27, R51 to R28, R52 to R29, R7 to R8, R10 to R9, SW4 to SW2, SW2 to SW3, SW3 to SW4

Commit message: New buck I think
Trying to make buck work
Parts:
- D10, D11, D2, D3, D4, D5, D6, D7, D8, D9: footprint (none) -> LED_SMD:LED_0603_1608Metric_Pad1.05x0.95mm_HandSolder
- R10, R11, R12, R13, R14, R15, R16, R17, R18, R19, R20, R21, R22, R23, R24, R25, R26, R27, R28, R8, R9: footprint (none) -> Resistor_SMD:R_0603_1608Metric_Pad0.98x0.95mm_HandSolder
- R29: footprint (none) -> Resistor_SMD:R_0201_0603Metric_Pad0.64x0.40mm_HandSolder
Changed lines of the file:
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@@
 			)
 		)
-		(property "Footprint" ""
+		(property "Footprint" "LED_SMD:LED_0603_1608Metric_Pad1.05x0.95mm_HandSolder"
 			(at 184.15 34.29 0)
 			(hide yes)
@@
 			)
 		)
-		(property "Footprint" ""
+		(property "Footprint" "LED_SMD:LED_0603_1608Metric_Pad1.05x0.95mm_HandSolder"
 			(at 107.95 69.85 0)
 			(hide yes)
@@
 			)
 		)
-		(property "Footprint" ""
+		(property "Footprint" "LED_SMD:LED_0603_1608Metric_Pad1.05x0.95mm_HandSolder"
 			(at 241.3 33.02 0)
 			(hide yes)
@@
 			)
 		)
-		(property "Footprint" ""
+		(property "Footprint" "LED_SMD:LED_0603_1608Metric_Pad1.05x0.95mm_HandSolder"
 			(at 41.91 67.31 0)
 			(hide yes)
@@
 			)
 		)
-		(property "Footprint" ""
+		(property "Footprint" "LED_SMD:LED_0603_1608Metric_Pad1.05x0.95mm_HandSolder"
 			(at 74.93 91.44 0)
 			(hide yes)
@@
 			)
 		)
-		(property "Footprint" ""
+		(property "Footprint" "Resistor_SMD:R_0603_1608Metric_Pad0.98x0.95mm_HandSolder"
 			(at 185.166 43.434 90)
 			(hide yes)
@@
 			)
 		)
-		(property "Footprint" ""
+		(property "Footprint" "Resistor_SMD:R_0603_1608Metric_Pad0.98x0.95mm_HandSolder"
 			(at 116.586 143.764 90)
 			(hide yes)
@@
 			)
 		)
-		(property "Footprint" ""
+		(property "Footprint" "Resistor_SMD:R_0603_1608Metric_Pad0.98x0.95mm_HandSolder"
 			(at 170.434 52.324 90)
 			(hide yes)
@@
 			)
 		)
-		(property "Footprint" ""
+		(property "Footprint" "Resistor_SMD:R_0603_1608Metric_Pad0.98x0.95mm_HandSolder"
 			(at 87.376 46.736 90)
 			(hide yes)
@@
 			)
 		)
-		(property "Footprint" ""
+		(property "Footprint" "Resistor_SMD:R_0603_1608Metric_Pad0.98x0.95mm_HandSolder"
 			(at 138.176 124.714 90)
 			(hide yes)
@@
 			)
 		)
-		(property "Footprint" ""
+		(property "Footprint" "LED_SMD:LED_0603_1608Metric_Pad1.05x0.95mm_HandSolder"
 			(at 137.16 115.57 0)
 			(hide yes)
@@
 			)
 		)
-		(property "Footprint" ""
+		(property "Footprint" "Resistor_SMD:R_0603_1608Metric_Pad0.98x0.95mm_HandSolder"
 			(at 167.386 109.474 90)
 			(hide yes)
@@
 			)
 		)
-		(property "Footprint" ""
+		(property "Footprint" "Resistor_SMD:R_0603_1608Metric_Pad0.98x0.95mm_HandSolder"
 			(at 242.316 42.164 90)
 			(hide yes)
@@
 			)
 		)
-		(property "Footprint" ""
+		(property "Footprint" "Resistor_SMD:R_0603_1608Metric_Pad0.98x0.95mm_HandSolder"
 			(at 214.884 138.684 90)
 			(hide yes)
@@
 			)
 		)
-		(property "Footprint" ""
+		(property "Footprint" "Resistor_SMD:R_0603_1608Metric_Pad0.98x0.95mm_HandSolder"
 			(at 51.816 68.326 90)
 			(hide yes)
@@
 			)
 		)
-		(property "Footprint" ""
+		(property "Footprint" "LED_SMD:LED_0603_1608Metric_Pad1.05x0.95mm_HandSolder"
 			(at 267.97 77.47 0)
 			(hide yes)
@@
 			)
 		)
-		(property "Footprint" ""
+		(property "Footprint" "Resistor_SMD:R_0603_1608Metric_Pad0.98x0.95mm_HandSolder"
 			(at 220.726 61.214 90)
 			(hide yes)
@@
 			)
 		)
-		(property "Footprint" ""
+		(property "Footprint" "Resistor_SMD:R_0603_1608Metric_Pad0.98x0.95mm_HandSolder"
 			(at 208.026 148.844 90)
 			(hide yes)
@@
 			)
 		)
-		(property "Footprint" ""
+		(property "Footprint" "Resistor_SMD:R_0201_0603Metric_Pad0.64x0.40mm_HandSolder"
 			(at 268.986 86.614 90)
 			(hide yes)
@@
 			)
 		)
-		(property "Footprint" ""
+		(property "Footprint" "Resistor_SMD:R_0603_1608Metric_Pad0.98x0.95mm_HandSolder"
 			(at 188.976 90.424 90)
 			(hide yes)
@@
 			)
 		)
-		(property "Footprint" ""
+		(property "Footprint" "LED_SMD:LED_0603_1608Metric_Pad1.05x0.95mm_HandSolder"
 			(at 77.47 45.72 0)
 			(hide yes)
@@
 			)
 		)
-		(property "Footprint" ""
+		(property "Footprint" "Resistor_SMD:R_0603_1608Metric_Pad0.98x0.95mm_HandSolder"
 			(at 123.444 133.604 90)
 			(hide yes)
@@
 			)
 		)
-		(property "Footprint" ""
+		(property "Footprint" "Resistor_SMD:R_0603_1608Metric_Pad0.98x0.95mm_HandSolder"
 			(at 227.584 51.054 90)
 			(hide yes)
@@
 			)
 		)
-		(property "Footprint" ""
+		(property "Footprint" "Resistor_SMD:R_0603_1608Metric_Pad0.98x0.95mm_HandSolder"
 			(at 254.254 95.504 90)
 			(hide yes)
@@
 			)
 		)
-		(property "Footprint" ""
+		(property "Footprint" "Resistor_SMD:R_0603_1608Metric_Pad0.98x0.95mm_HandSolder"
 			(at 84.836 92.456 90)
 			(hide yes)
@@
 			)
 		)
-		(property "Footprint" ""
+		(property "Footprint" "LED_SMD:LED_0603_1608Metric_Pad1.05x0.95mm_HandSolder"
 			(at 228.6 120.65 0)
 			(hide yes)
@@
 			)
 		)
-		(property "Footprint" ""
+		(property "Footprint" "Resistor_SMD:R_0603_1608Metric_Pad0.98x0.95mm_HandSolder"
 			(at 229.616 129.794 90)
 			(hide yes)
@@
 			)
 		)
-		(property "Footprint" ""
+		(property "Footprint" "Resistor_SMD:R_0603_1608Metric_Pad0.98x0.95mm_HandSolder"
 			(at 247.396 105.664 90)
 			(hide yes)
@@
 			)
 		)
-		(property "Footprint" ""
+		(property "Footprint" "Resistor_SMD:R_0603_1608Metric_Pad0.98x0.95mm_HandSolder"
 			(at 174.244 99.314 90)
 			(hide yes)
@@
 			)
 		)
-		(property "Footprint" ""
+		(property "Footprint" "LED_SMD:LED_0603_1608Metric_Pad1.05x0.95mm_HandSolder"
 			(at 187.96 81.28 0)
 			(hide yes)
@@
 			)
 		)
-		(property "Footprint" ""
+		(property "Footprint" "Resistor_SMD:R_0603_1608Metric_Pad0.98x0.95mm_HandSolder"
 			(at 117.856 70.866 90)
 			(hide yes)
@@
 			)
 		)
-		(property "Footprint" ""
+		(property "Footprint" "Resistor_SMD:R_0603_1608Metric_Pad0.98x0.95mm_HandSolder"
 			(at 163.576 62.484 90)
 			(hide yes)

Commit message: Almost done with Schematic
Parts:
- R29: footprint Resistor_SMD:R_0201_0603Metric_Pad0.64x0.40mm_HandSolder -> Resistor_SMD:R_0603_1608Metric_Pad0.98x0.95mm_HandSolder
- SW1, SW2, SW3, SW4: footprint (none) -> MRDT_Switches:SW_SPST_TL3305A
Changed lines of the file:
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@@
 			)
 		)
-		(property "Footprint" ""
+		(property "Footprint" "MRDT_Switches:SW_SPST_TL3305A"
 			(at 109.22 77.47 0)
 			(hide yes)
@@
 			)
 		)
-		(property "Footprint" ""
+		(property "Footprint" "MRDT_Switches:SW_SPST_TL3305A"
 			(at 78.74 53.34 0)
 			(hide yes)
@@
 			)
 		)
-		(property "Footprint" "Resistor_SMD:R_0201_0603Metric_Pad0.64x0.40mm_HandSolder"
+		(property "Footprint" "Resistor_SMD:R_0603_1608Metric_Pad0.98x0.95mm_HandSolder"
 			(at 268.986 86.614 90)
 			(hide yes)
@@
 			)
 		)
-		(property "Footprint" ""
+		(property "Footprint" "MRDT_Switches:SW_SPST_TL3305A"
 			(at 43.18 74.93 0)
 			(hide yes)
@@
 			)
 		)
-		(property "Footprint" ""
+		(property "Footprint" "MRDT_Switches:SW_SPST_TL3305A"
 			(at 76.2 99.06 0)
 			(hide yes)

Commit message: Layout updates
footprint changes
Parts:
- S1: footprint CoreBoard:DIPS762W56P254L991H597Q6N -> 94HBBBO6T:DIPS762W56P254L991H597Q6N
Changed lines of the file:
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@@
 			)
 		)
-		(property "Footprint" "CoreBoard:DIPS762W56P254L991H597Q6N"
+		(property "Footprint" "94HBBBO6T:DIPS762W56P254L991H597Q6N"
 			(at 53.34 229.54 0)
 			(hide yes)

Commit message: add pan right led
Parts:
- added D13: Blue, LED_SMD:LED_0603_1608Metric_Pad1.05x0.95mm_HandSolder, symbol Device:LED
- added Q8: BSS138, Package_TO_SOT_SMD:SOT-23, symbol Transistor_FET:BSS138
- added R32: 10k, Resistor_SMD:R_0603_1608Metric_Pad0.98x0.95mm_HandSolder, symbol Device:R_US
- added R33: 100, Resistor_SMD:R_0603_1608Metric_Pad0.98x0.95mm_HandSolder, symbol Device:R_US
- added R37: 1k, Resistor_SMD:R_0603_1608Metric_Pad0.98x0.95mm_HandSolder, symbol Device:R_US
Connections:
- net +3V3: now also D13.2 (A)
- net GND: now also Q8.2 (S), R32.2
- net PanRight_LED: now also R32.1, R33.1
- new net: D13.1 (K), R37.1
- new net: Q8.3 (D), R37.2
- new net: Q8.1 (G), R33.2
